Commit message: change joint name

File: jaco_model/urdf/no_finger.urdf (robot description, URDF)
Before this commit: robot jaco, 11 links, 10 joints
Links:
- removed link jaco_link_finger_1
- removed link jaco_link_finger_2
- removed link jaco_link_finger_3
Joints:
- removed joint jaco_joint_finger_1
- removed joint jaco_joint_finger_2
- removed joint jaco_joint_finger_3

File: jaco_model/urdf/no_finger_alone.xacro (robot description, xacro)
@@ -13,5 +13,5 @@
     xmlns:physics="http://playerstage.sourceforge.net/gazebo/xmlschema/#physics"
 xmlns:xacro="http://ros.org/wiki/xacro" name="jaco">
-  <xacro:include filename="$(find jaco_model)/urdf/jaco_arm.xacro" />
+  <xacro:include filename="$(find jaco_model)/urdf/no_finger.xacro" />
 <link name="root">
       <visual>
