Commit message: Update standalone_arm.urdf

File: jaco_model/urdf/standalone_arm.urdf (robot description, URDF)
Before this commit: robot jaco, 11 links, 10 joints
Joints:
- joint jaco_joint_1: axis 0 0 1 -> 0 0 -1; origin xyz=0 0 0.1535 rpy=3.14159265359 0 0 -> xyz=0 0 0.1535 rpy=3.14159265359 0 3.14159265359
- joint jaco_joint_2: origin xyz=0 0 -0.1185 rpy=-1.57079632679 -1.57079632679 0 -> xyz=0 0 -0.1185 rpy=-1.57079632679 3.14159265359 0
- joint jaco_joint_3: axis 0 0 1 -> 0 0 -1; origin xyz=0.41 0 0 rpy=3.14159265359 0 3.14159265359 -> xyz=0.41 0 0 rpy=3.14159265359 0 1.57079632679
- joint jaco_joint_4: axis 0 0 1 -> 0 0 -1; origin xyz=0.207 0 -0.01125 rpy=0 -1.57079632679 0 -> xyz=0.207 0 -0.01125 rpy=3.14159265359 1.57079632679 0
- joint jaco_joint_5: axis 0 0 1 -> 0 0 -1; origin xyz=0.0343 0 -0.06588 rpy=0 0.959931088597 3.14159265359 -> xyz=0.0343 0 -0.06588 rpy=0 -0.959931088597 0
- joint jaco_joint_6: axis 0 0 1 -> 0 0 -1; origin xyz=0.0343 0 -0.06588 rpy=0 0.959931088597 3.14159265359 -> xyz=0.0343 0 -0.06588 rpy=-0.959931088597 0 1.57079632679
